Commit message: ver. 3

File: rcm/urdf/rcm.urdf (robot description, URDF)
Before this commit: robot rcm, 11 links, 7 joints
Links:
- link Link1: mass 0.340818102148623 -> 0.34082
- link Link3_1: mass 0.0439955519370354 -> 0.043996
- link Link3_2: mass 0.0439955519370354 -> 0.043996
- link Link_ee: mass 0.0923069522797063 -> 0.092307
- link Link_ee_: mass 0.0857843743614275 -> 0.085784
Joints:
- added joint Link3_1_joint_: type revolute, parent Link2_2, child Link3_1_, origin xyz=0.072 0 0 rpy=0 0 -1.5708, axis 0 0 1, limit lower=-10 upper=10 effort=10 velocity=10
- added joint Link3_2_joint_: type revolute, parent Link2_2, child Link3_2_, origin xyz=0.112 0 0 rpy=0 0 -1.5708, axis 0 0 1, limit lower=-10 upper=10 effort=10 velocity=10
- added joint Link_ee_joint_: type revolute, parent Link3_2, child Link_ee_, origin xyz=0.1675 0 0 rpy=0 0 -1.5708, axis 0 0 1, limit lower=-10 upper=10 effort=10 velocity=10
- joint Link3_1_joint: child Link3_1_ -> Link3_1; parent Link2_2 -> Link2_1
- joint Link3_2_joint: child Link3_2_ -> Link3_2; mimic (none) -> joint=Link3_1_joint multiplier=1 offset=0; parent Link2_2 -> Link2_1
- joint Link_ee_joint: child Link_ee_ -> Link_ee; parent Link3_2 -> Link3_1

Commit message: ver.4

File: rcm/urdf/rcm.urdf (robot description, URDF)
Before this commit: robot rcm, 11 links, 10 joints
Links:
- removed link Link3_1_
- removed link Link3_2_
- removed link Link_ee_
- link base_link: mass 0.548884585225384 -> 0.54888
Joints:
- removed joint Link3_1_joint_
- removed joint Link3_2_joint_
- removed joint Link_ee_joint_
- joint Link_E_joint: limit lower=-10 upper=10 effort=10 velocity=10 -> lower=-0.03 upper=0.04 effort=10 velocity=10; origin xyz=-0.0074884 -0.037 0 rpy=1.5708 0 1.5381 -> xyz=0.032512 -0.037 0 rpy=1.5708 0 1.5381
- joint Link_ee_joint: origin xyz=0.1675 0 0 rpy=0 0 -1.5708 -> xyz=0.1675 0.04 0 rpy=0 0 -1.5708

Commit message: sdf

File: rcm/urdf/rcm.urdf (robot description, URDF)
Before this commit: robot rcm, 8 links, 7 joints
Joints:
- joint Link2_1_joint: mimic joint=Link2_1_joint multiplier=1 offset=0 -> (none)
